Commit message: update and works

File: urdf/delta_admittance_demo.urdf.xacro (robot description, xacro)
@@ -4,5 +4,5 @@
   <xacro:property name="use_fake_hardware" value="true" />
   <!-- Base link (world frame) -->
-  <link name="base">
+  <link name="base_link">
     <inertial>
       <mass value="10.0"/>
@@ -25,5 +25,5 @@
   <!-- Joint 1 (0 degrees) -->
   <joint name="joint1" type="revolute">
-    <parent link="base"/>
+    <parent link="base_link"/>
     <child link="upper_arm_1"/>
     <origin xyz="${base_radius} 0 ${motor_offset}" rpy="0 0 0"/>
@@ -49,5 +49,5 @@
   <!-- Joint 2 (120 degrees) -->
   <joint name="joint2" type="revolute">
-    <parent link="base"/>
+    <parent link="base_link"/>
     <child link="upper_arm_2"/>
     <origin xyz="${-base_radius*0.5} ${base_radius*0.866} ${motor_offset}" rpy="0 0 ${2*pi/3}"/>
@@ -73,5 +73,5 @@
   <!-- Joint 3 (240 degrees) -->
   <joint name="joint3" type="revolute">
-    <parent link="base"/>
+    <parent link="base_link"/>
     <child link="upper_arm_3"/>
     <origin xyz="${-base_radius*0.5} ${-base_radius*0.866} ${motor_offset}" rpy="0 0 ${4*pi/3}"/>
@@ -119,6 +119,5 @@
     <axis xyz="0 1 0"/>
   </joint>
-  <link name="lower_link_1"/>
-  <link name="lower_link_vis_1">
+  <link name="lower_link_1">
     <visual>
       <geometry>
@@ -137,9 +136,4 @@
     <axis xyz="0 0 1"/>
   </joint>
-  <joint name="lower_link_vis_joint_1" type="fixed">
-    <parent link="lower_pitch_link_1"/>
-    <child link="lower_link_vis_1"/>
-    <origin xyz="0 0 0" rpy="0 0 0"/>
-  </joint>
   <link name="lower_arm_end_1">
     <visual>
@@ -153,5 +147,5 @@
   </link>
   <joint name="lower_arm_end_joint_1" type="fixed">
-    <parent link="lower_link_vis_1"/>
+    <parent link="lower_link_1"/>
     <child link="lower_arm_end_1"/>
     <origin xyz="-0.34 0 0" rpy="0 0 0"/>
@@ -180,6 +174,5 @@
     <axis xyz="0 1 0"/>
   </joint>
-  <link name="lower_link_2"/>
-  <link name="lower_link_vis_2">
+  <link name="lower_link_2">
     <visual>
       <geometry>
@@ -198,9 +191,4 @@
     <axis xyz="0 0 1"/>
   </joint>
-  <joint name="lower_link_vis_joint_2" type="fixed">
-    <parent link="lower_pitch_link_2"/>
-    <child link="lower_link_vis_2"/>
-    <origin xyz="0 0 0" rpy="0 0 0"/>
-  </joint>
   <link name="lower_arm_end_2">
     <visual>
@@ -214,5 +202,5 @@
   </link>
   <joint name="lower_arm_end_joint_2" type="fixed">
-    <parent link="lower_link_vis_2"/>
+    <parent link="lower_link_2"/>
     <child link="lower_arm_end_2"/>
     <origin xyz="-0.34 0 0" rpy="0 0 0"/>
@@ -241,6 +229,5 @@
     <axis xyz="0 1 0"/>
   </joint>
-  <link name="lower_link_3"/>
-  <link name="lower_link_vis_3">
+  <link name="lower_link_3">
     <visual>
       <geometry>
@@ -259,9 +246,4 @@
     <axis xyz="0 0 1"/>
   </joint>
-  <joint name="lower_link_vis_joint_3" type="fixed">
-    <parent link="lower_pitch_link_3"/>
-    <child link="lower_link_vis_3"/>
-    <origin xyz="0 0 0" rpy="0 0 0"/>
-  </joint>
   <link name="lower_arm_end_3">
     <visual>
@@ -275,5 +257,5 @@
   </link>
   <joint name="lower_arm_end_joint_3" type="fixed">
-    <parent link="lower_link_vis_3"/>
+    <parent link="lower_link_3"/>
     <child link="lower_arm_end_3"/>
     <origin xyz="-0.34 0 0" rpy="0 0 0"/>
@@ -296,9 +278,9 @@
     </visual>
   </link>
-  <!-- Floating joint for end effector (managed by delta kinematics controller) -->
+  <!-- Floating joint: the delta kinematics controller broadcasts
+       the true base_link→end_effector transform on /tf at runtime. -->
   <joint name="ee_floating" type="floating">
-    <parent link="base"/>
+    <parent link="base_link"/>
     <child link="end_effector"/>
-    <origin xyz="0 0 -0.4" rpy="0 0 0"/>
   </joint>
   <!-- ros2_control configuration -->

File: urdf/delta_robot.urdf.xacro (robot description, xacro)
@@ -10,5 +10,5 @@
   <xacro:property name="delta_motor_z_offset" value="-0.025"/>
   <!-- Base link -->
-  <link name="base">
+  <link name="base_link">
     <visual>
       <geometry>
@@ -18,4 +18,10 @@
       <material name="gray"><color rgba="0.6 0.6 0.6 1.0"/></material>
     </visual>
+    <collision>
+      <geometry>
+        <cylinder length="0.02" radius="0.06"/>
+      </geometry>
+      <origin xyz="0 0 ${delta_motor_z_offset}" rpy="0 0 0"/>
+    </collision>
   </link>
   <!-- Three simple revolute joints and arms for visualization -->
@@ -31,7 +37,13 @@
         <material name="blue"><color rgba="0.2 0.4 0.8 1.0"/></material>
       </visual>
+      <collision>
+        <geometry>
+          <cylinder length="${delta_rf}" radius="0.01"/>
+        </geometry>
+        <origin xyz="${delta_rf/2.0} 0 0" rpy="0 ${pi/2} 0"/>
+      </collision>
     </link>
     <joint name="joint${idx}" type="revolute">
-      <parent link="base"/>
+      <parent link="base_link"/>
       <child link="upper_link_${idx}"/>
       <!-- Rotate around local Y axis (perpendicular to radial direction)
@@ -50,4 +62,9 @@
         <material name="gray"><color rgba="0.5 0.5 0.5 1.0"/></material>
       </visual>
+      <collision>
+        <geometry>
+          <sphere radius="0.015"/>
+        </geometry>
+      </collision>
     </link>
     <joint name="elbow_joint_${idx}" type="fixed">
@@ -67,8 +84,4 @@
     <!-- Lower arm (forearm, connected to end-effector via ball joint) -->
     <link name="lower_link_${idx}">
-      <!-- Physical lower link (no visual) - visual geometry moved to lower_link_vis for controller-driven TF visualization -->
-    </link>
-    <!-- Visual-only lower arm link (driven by controller TF) -->
-    <link name="lower_link_vis_${idx}">
       <visual>
         <geometry>
@@ -79,4 +92,10 @@
         <material name="green"><color rgba="0.2 0.8 0.4 1.0"/></material>
       </visual>
+      <collision>
+        <geometry>
+          <cylinder length="${delta_re}" radius="0.008"/>
+        </geometry>
+        <origin xyz="${-delta_re/2.0} 0 0" rpy="0 ${pi/2} 0"/>
+      </collision>
     </link>
     <!-- Ball joint yaw: rotation around Z axis (after pitch) -->
@@ -87,10 +106,4 @@
       <axis xyz="0 0 1"/>  <!-- Yaw around Z axis (after pitch rotation) -->
     </joint>
-    <!-- Visual-only lower link fixed to the pitch link; its transform will be published by the controller -->
-    <joint name="lower_link_vis_joint_${idx}" type="fixed">
-      <parent link="lower_pitch_link_${idx}"/>
-      <child link="lower_link_vis_${idx}"/>
-      <origin xyz="0 0 0" rpy="0 0 0"/>
-    </joint>
     <!-- End point of lower arm (where it attaches to EE platform) -->
     <link name="lower_arm_end_${idx}">
@@ -101,7 +114,12 @@
         <material name="gray"><color rgba="0.5 0.5 0.5 1.0"/></material>
       </visual>
+      <collision>
+        <geometry>
+          <sphere radius="0.012"/>
+        </geometry>
+      </collision>
     </link>
     <joint name="lower_arm_end_joint_${idx}" type="fixed">
-      <parent link="lower_link_vis_${idx}"/>
+      <parent link="lower_link_${idx}"/>
       <child link="lower_arm_end_${idx}"/>
       <origin xyz="${-delta_re} 0 0" rpy="0 0 0"/>  <!-- At the end of the lower arm (in -X direction) -->
@@ -123,10 +141,16 @@
       <material name="red"><color rgba="0.8 0.2 0.2 1.0"/></material>
     </visual>
+    <collision>
+      <geometry>
+        <sphere radius="${delta_e}"/>
+      </geometry>
+    </collision>
   </link>
-  <!-- Floating joint allows ee to move freely in 6-DOF
-       The controller will publish the actual base→ee transform via TF -->
-  <joint name="ee_floating" type="floating">
-    <parent link="base"/>
+  <!-- Floating joint — robot_state_publisher ignores this;
+       the delta kinematics controller broadcasts the EE TF directly. -->
+  <joint name="ee_joint" type="floating">
+    <parent link="base_link"/>
     <child link="ee"/>
+    <origin xyz="0 0 0" rpy="0 0 0"/>
   </joint>
   <!-- Visual markers for EE platform attachment points (actual lower arm end positions) -->
